Commit message: Stabilize Gazebo MoveIt execution

File: src/ur_description/urdf/inc/ur_macro.xacro (robot description, xacro)
@@ -227,5 +227,5 @@
          <safety_controller soft_lower_limit="${shoulder_pan_lower_limit + safety_pos_margin}" soft_upper_limit="${shoulder_pan_upper_limit - safety_pos_margin}" k_position="${safety_k_position}" k_velocity="0.0"/>
       </xacro:if>
-      <dynamics damping="0" friction="0"/>
+      <dynamics damping="1.0" friction="0.1"/>
     </joint>
     <joint name="${prefix}shoulder_lift_joint" type="revolute">
@@ -239,5 +239,5 @@
          <safety_controller soft_lower_limit="${shoulder_lift_lower_limit + safety_pos_margin}" soft_upper_limit="${shoulder_lift_upper_limit - safety_pos_margin}" k_position="${safety_k_position}" k_velocity="0.0"/>
       </xacro:if>
-      <dynamics damping="0" friction="0"/>
+      <dynamics damping="1.0" friction="0.1"/>
     </joint>
     <joint name="${prefix}elbow_joint" type="revolute">
@@ -251,5 +251,5 @@
          <safety_controller soft_lower_limit="${elbow_joint_lower_limit + safety_pos_margin}" soft_upper_limit="${elbow_joint_upper_limit - safety_pos_margin}" k_position="${safety_k_position}" k_velocity="0.0"/>
       </xacro:if>
-      <dynamics damping="0" friction="0"/>
+      <dynamics damping="1.0" friction="0.1"/>
     </joint>
     <joint name="${prefix}wrist_1_joint" type="revolute">
@@ -263,5 +263,5 @@
          <safety_controller soft_lower_limit="${wrist_1_lower_limit + safety_pos_margin}" soft_upper_limit="${wrist_1_upper_limit - safety_pos_margin}" k_position="${safety_k_position}" k_velocity="0.0"/>
       </xacro:if>
-      <dynamics damping="0" friction="0"/>
+      <dynamics damping="1.0" friction="0.1"/>
     </joint>
     <joint name="${prefix}wrist_2_joint" type="revolute">
@@ -275,5 +275,5 @@
          <safety_controller soft_lower_limit="${wrist_2_lower_limit + safety_pos_margin}" soft_upper_limit="${wrist_2_upper_limit - safety_pos_margin}" k_position="${safety_k_position}" k_velocity="0.0"/>
       </xacro:if>
-      <dynamics damping="0" friction="0"/>
+      <dynamics damping="1.0" friction="0.1"/>
     </joint>
     <joint name="${prefix}wrist_3_joint" type="revolute">
@@ -287,5 +287,5 @@
          <safety_controller soft_lower_limit="${wrist_3_lower_limit + safety_pos_margin}" soft_upper_limit="${wrist_3_upper_limit - safety_pos_margin}" k_position="${safety_k_position}" k_velocity="0.0"/>
       </xacro:if>
-      <dynamics damping="0" friction="0"/>
+      <dynamics damping="1.0" friction="0.1"/>
     </joint>
     <!-- ROS-Industrial 'base' frame: base_link to UR 'Base' Coordinates transform -->

File: src/ur_description/urdf/ur3_dual_gazebo.xacro (robot description, xacro)
@@ -24,10 +24,4 @@
       </geometry>
     </visual>
-    <collision>
-      <origin xyz="0 0 0" rpy="0 0 0" />
-      <geometry>
-        <mesh filename="package://ur_description/meshes/base.stl" />
-      </geometry>
-    </collision>
    </link>
    <joint name="base_left" type="fixed">
